File: mcp_test.kicad_pcb (KiCad board)
At the start: 2 copper layers, 0 parts

Commit message: board: placed, routed, GND pours, DRC clean
Parts:
- added C1: 10uF, Capacitor_SMD:C_0805_2012Metric, F.Cu at (118.0, 118.2)
- added C2: 22uF Tant, Capacitor_Tantalum_SMD:CP_EIA-3528-21_Kemet-B, F.Cu at (132.0, 115.0)
- added D1: PWR, LED_SMD:LED_0805_2012Metric, F.Cu at (136.5, 120.0)
- added J1: USB-C Power, Connector_USB:USB_C_Receptacle_GCT_USB4125-xx-x-0190_6P_TopMnt_Horizontal, F.Cu at (104.0, 115.0)
- added R1: 5.1k, Resistor_SMD:R_0805_2012Metric, F.Cu at (112.0, 107.0)
- added R2: 5.1k, Resistor_SMD:R_0805_2012Metric, F.Cu at (112.0, 123.0)
- added R3: 1k, Resistor_SMD:R_0805_2012Metric, F.Cu at (136.5, 110.0)
- added U1: AMS1117-3.3, Package_TO_SOT_SMD:SOT-223-3_TabPin2, F.Cu at (125.0, 115.0)
Routing:
- net VBUS: track 0.00 -> 20.6 mm
- net +3V3: track 0.00 -> 19.0 mm
- net GND: track 0.00 -> 15.0 mm, vias 0 -> 6
- net CC2: track 0.00 -> 9.34 mm, vias 0 -> 2
- net CC1: track 0.00 -> 9.34 mm, vias 0 -> 2
- net LED_A: track 0.00 -> 8.15 mm
- added copper zone on B.Cu, net GND
- added copper zone on F.Cu, net GND
Other:
- board outline added: 40 x 30 mm
