File: mcp_test.kicad_sch (KiCad schematic)
At the start: 8 parts, among them J1 USB-C Power, U1 AMS1117-3.3

Commit message: board: placed, routed, GND pours, DRC clean
Parts:
- J1: footprint (none) -> Connector_USB:USB_C_Receptacle_GCT_USB4125-xx-x-0190_6P_TopMnt_Horizontal; MPN (none) -> USB4125-GF-A-0190; Manufacturer (none) -> GCT
Changed lines of the file:
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@@
 			)
 		)
-		(property "Footprint" ""
+		(property "Footprint" "Connector_USB:USB_C_Receptacle_GCT_USB4125-xx-x-0190_6P_TopMnt_Horizontal"
 			(at 63.5 102.87 0)
 			(hide yes)
@@
 			)
 		)
+    (property "MPN" "USB4125-GF-A-0190" (at 59.69 100.33 0)
+      (effects (font (size 1.27 1.27)) (hide yes))
+    )
+    (property "Manufacturer" "GCT" (at 59.69 100.33 0)
+      (effects (font (size 1.27 1.27)) (hide yes))
+    )
 		(pin "A12"
 		)
